File: FGINT-V4-MASTER-128/FGINT-V4-MASTER-128.sch (KiCad schematic (older format))
At the start: 68 parts, among them J1 OUT1-16, J10 ComGPIOB1, J11 ComGPIOA5, J12 ComGPIOB5, J13 OUT33-48, J14 OUT97-112, J15 ComGPIOA2, J16 ComGPIOB2, J17 ComGPIOA6, J18 ComGPIOB6, J19 OUT48-64, J2 OUT65-80, J20 OUT112-128, J21 ComGPIOA3, J22 ComGPIOB3, J23 ComGPIOA7, J24 ComGPIOB7, J25 9V DC, J26 Raspberry, J27 PC Power Input, J28 Exp01, J29 Expd02, J3 ComGPIOA0, J30 Expd03, J31 Exp04, J4 ComGPIOB0, J5 ComGPIOA4, J6 ComGPIOB4, J7 OUT17-32, J8 OUT81-96, J9 ComGPIOA1, Q1 2N7000, Q2 2N7000, U1 MCP23017_SP, U10 LM317_3PinPackage, U2 MCP23017_SP, U3 MCP23017_SP, U4 MCP23017_SP, U5 MCP23017_SP, U6 MCP23017_SP, U7 MCP23017_SP, U8 MCP23017_SP, U9 LM7805_TO220

Commit message: Update Power with +12V on Screw header
Parts:
- removed J27: PC Power Input, TerminalBlock:TerminalBlock_bornier-3_P5.08mm, symbol Connector:Screw_Terminal_01x03
- added J27: 3.3 ENBL, Connector_PinHeader_2.54mm:PinHeader_1x02_P2.54mm_Vertical, symbol Connector_Generic:Conn_01x02
- added J32: 5VPI, Connector_PinHeader_2.54mm:PinHeader_1x02_P2.54mm_Vertical, symbol Connector_Generic:Conn_01x02
- added J33: PC Power Input, TerminalBlock:TerminalBlock_bornier-4_P5.08mm, symbol Connector:Screw_Terminal_01x04
- J25: value 9V DC -> 9V - 12V DC
- RN1, RN10, RN11, RN12, RN13, RN14, RN15, RN16, RN2, RN3, RN4, RN5, RN6, RN7, RN8, RN9: value R_Network08 -> 10K
- U10: value LM317_3PinPackage -> LM317
- U9: value LM7805_TO220 -> LM7805
Connections:
- net +3V3: now also J33.2 (Pin_2)
- net +9V: now also J27.2 (Pin_2), J33.1 (Pin_1); no longer U10.3 (VI)
- net GND: now also J33.4 (Pin_4)
- net INTA0: now also J26.35 (Pin_35); no longer J26.13 (Pin_13)
- net INTA1: now also J26.31 (Pin_31); no longer J26.29 (Pin_29)
- net INTA2: now also J26.15 (Pin_15); no longer J26.33 (Pin_33)
- net INTA3: now also J26.11 (Pin_11); no longer J26.37 (Pin_37)
- net INTB0: now also J26.37 (Pin_37); no longer J26.11 (Pin_11)
- net INTB1: now also J26.33 (Pin_33); no longer J26.15 (Pin_15)
- net INTB2: now also J26.29 (Pin_29); no longer J26.31 (Pin_31)
- net INTB3: now also J26.13 (Pin_13); no longer J26.35 (Pin_35)
- net +5VPIB: now reaches J26.2 (Pin_2)
- net +5VPIB: now also J26.4 (Pin_4), J32.1 (Pin_1)
- new net +5VPIA: J32.2 (Pin_2), J33.3 (Pin_3)
- new net ENBL3.3: J27.1 (Pin_1), U10.3 (VI)
- no-connect marks 0 -> 12
Other:
- moved on the sheet: C1, C2, C3, J25, R3, R6, U10, U9
